File: osu_keypad_version_2.0/osu_keypad_version_2.0.kicad_sch (KiCad schematic)
At the start: 14 parts, among them SW1 SW_Push, U1 ATmega32U4-A, Y1 16Mhz

Commit message: finished part 4 of ai03's guide
Parts:
- added D1, D2, D3, D4: SOD-123, Diode_SMD:D_SOD-123, symbol Device:D_Small
- added F1: 500mA, Fuse:Fuse_1206_3216Metric, symbol Device:Polyfuse_Small
- added MX1, MX2, MX3, MX4: MX-NoLED, MX_Alps_Hybrid:MX-1U-NoLED, symbol MX_Alps_Hybrid:MX-NoLED
- added USB2: Molex-0548190589, random-keyboard-parts:Molex-0548190589, symbol random-keyboard-parts:Molex-0548190589
- C1, C2, C3, C4, C5, C6, C7: footprint (none) -> Capacitor_SMD:C_0805_2012Metric
- R1, R2, R3, R4: footprint (none) -> Resistor_SMD:R_0805_2012Metric
- SW1: footprint (none) -> random-keyboard-parts:SKQG-1155865
- Y1: footprint (none) -> Crystal:Crystal_SMD_3225-4Pin_3.2x2.5mm
Connections:
- net +5V: now also F1.2
- net D+: now also USB2.3 (D+)
- net D-: now also USB2.4 (D-)
- net GND: now also USB2.1 (GND)
- new net: D2.2 (A), MX2.2 (ROW)
- new net: D3.2 (A), MX3.2 (ROW)
- new net: D1.2 (A), MX1.2 (ROW)
- new net: D4.2 (A), MX4.2 (ROW)
- new net COL 0: MX1.1 (COL), MX3.1 (COL)
- new net COL 1: MX2.1 (COL), MX4.1 (COL)
- new net ROW 0: D1.1 (K), D2.1 (K)
- new net ROW 1: D3.1 (K), D4.1 (K)
- new net VCC: F1.1, USB2.5 (VBUS)
Other:
- moved on the sheet: C1, C2, C3, C4, C5, C6, C7, R1, R2, R3, R4, SW1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

Commit message: routing done
Connections:
- net COL 0: now also U1.29 (PB5)
- net COL 1: now also U1.28 (PB4)
- net ROW 0: now also U1.27 (PD7)
- net ROW 1: now also U1.30 (PB6)
Changed lines of the file:
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@@
+    )
+  )
+  (global_label "ROW 0" (shape input) (at 114.3 109.22 0) (fields_autoplaced)
+    (effects (font (size 1.27 1.27)) (justify left))
+    (property "Intersheetrefs" "${INTERSHEET_REFS}" (at 123.5142 109.22 0)
+      (effects (font (size 1.27 1.27)) (justify left) hide)
     )
   )
@@
       (effects (font (size 1.27 1.27)) (justify left) hide)
     )
+  )
+  (global_label "ROW 1" (shape input) (at 114.3 76.2 0) (fields_autoplaced)
+    (effects (font (size 1.27 1.27)) (justify left))
+    (property "Intersheetrefs" "${INTERSHEET_REFS}" (at 123.5142 76.2 0)
+      (effects (font (size 1.27 1.27)) (justify left) hide)
+    )
+  )
+  (global_label "COL 0" (shape input) (at 114.3 73.66 0) (fields_autoplaced)
+    (effects (font (size 1.27 1.27)) (justify left))
+    (property "Intersheetrefs" "${INTERSHEET_REFS}" (at 123.0909 73.66 0)
+      (effects (font (size 1.27 1.27)) (justify left) hide)
+    )
+  )
+  (global_label "COL 1" (shape input) (at 114.3 71.12 0) (fields_autoplaced)
+    (effects (font (size 1.27 1.27)) (justify left))
+    (property "Intersheetrefs" "${INTERSHEET_REFS}" (at 123.0909 71.12 0)
+      (effects (font (size 1.27 1.27)) (justify left) hide)
+    )
